Commit message: Changing robot shapes

File: ball_pusher_robot/urdf/ball_pusher.urdf (robot description, URDF)
Before this commit: robot ball_pusher, 11 links, 10 joints
Links:
- removed link front_right_wheel
- removed link left_gripper_2
- removed link rear_left_wheel
- removed link rear_right_wheel
- removed link right_gripper_1
- removed link right_gripper_2
- link base_link: mass None -> 5.0; geometry collision box size=0.6 0.4 0.2; visual box size=0.6 0.4 0.2
- link front_left_wheel: mass None -> 0.5; geometry collision cylinder length=0.04 radius=0.08; visual cylinder length=0.04 radius=0.08
- link left_arm: mass None -> 0.3; geometry collision box size=0.45 0.05 0.1; visual box size=0.45 0.05 0.1
- link left_gripper_1: mass None -> 0.05; geometry collision box size=0.02 0.23 0.1; visual box size=0.02 0.23 0.1
- link right_arm: mass None -> 0.3; geometry collision box size=0.45 0.05 0.1; visual box size=0.45 0.05 0.1
Joints:
- removed joint front_right_wheel_joint
- removed joint left_gripper_2_joint
- removed joint rear_left_wheel_joint
- removed joint rear_right_wheel_joint
- removed joint right_gripper_1_joint
- removed joint right_gripper_2_joint
- joint left_arm_joint: axis 0 0 1 -> (none); limit lower=-1.2 upper=0.3 effort=10 velocity=1 -> (none); type revolute -> fixed
- joint left_gripper_1_joint: axis 0 -1 0 -> (none); limit lower=0 upper=0.08 effort=5 velocity=0.1 -> (none); type prismatic -> fixed
- joint right_arm_joint: axis 0 0 -1 -> (none); limit lower=-1.2 upper=0.3 effort=10 velocity=1 -> (none); type revolute -> fixed
