Commit message: Robot spawning success

File: ball_pusher_robot/urdf/ball_pusher_with_physics.urdf (robot description, URDF)
Before this commit: robot ball_pusher, 7 links, 6 joints
Links:
- added link left_gripper_2, mass 0.03; collision box size=0.02 0.12 0.1; visual box size=0.02 0.12 0.1
- added link right_arm, mass 0.3; collision box size=0.45 0.04 0.08; visual box size=0.45 0.05 0.1
- added link right_gripper_1, mass 0.05; collision box size=0.02 0.24 0.1; visual box size=0.02 0.24 0.1
- added link right_gripper_2, mass 0.03; collision box size=0.02 0.12 0.1; visual box size=0.02 0.12 0.1
- link left_arm: geometry collision box size=0.45 0.04 0.08; visual box size=0.45 0.05 0.1
Joints:
- added joint left_gripper_2_joint: type prismatic, parent left_arm, child left_gripper_2, origin xyz=0.20 0.06 0 rpy=0 0 0, axis 0 -1 0, limit lower=0 upper=0.08 effort=5 velocity=0.1
- added joint right_arm_joint: type revolute, parent base_link, child right_arm, origin xyz=0.35 -0.22 0.0 rpy=0 0 0, axis 0 0 -1, limit lower=-1.2 upper=0.3 effort=10 velocity=1
- added joint right_gripper_1_joint: type prismatic, parent right_arm, child right_gripper_1, origin xyz=0.20 0 0 rpy=0 0 0, axis 0 1 0, limit lower=0 upper=0.08 effort=5 velocity=0.1
- added joint right_gripper_2_joint: type prismatic, parent right_arm, child right_gripper_2, origin xyz=0.20 -0.06 0 rpy=0 0 0, axis 0 1 0, limit lower=0 upper=0.08 effort=5 velocity=0.1
- joint front_left_wheel_joint: origin xyz=0.2 0.22 -0.08 rpy=0 0 0 -> xyz=0.2 0.18 -0.08 rpy=0 0 0
- joint front_right_wheel_joint: origin xyz=0.2 -0.22 -0.08 rpy=0 0 0 -> xyz=0.2 -0.18 -0.08 rpy=0 0 0
- joint left_arm_joint: origin xyz=0.35 0.20 0.0 rpy=0 0 0 -> xyz=0.35 0.22 0.0 rpy=0 0 0
- joint rear_left_wheel_joint: origin xyz=-0.2 0.22 -0.08 rpy=0 0 0 -> xyz=-0.2 0.18 -0.08 rpy=0 0 0
- joint rear_right_wheel_joint: origin xyz=-0.2 -0.22 -0.08 rpy=0 0 0 -> xyz=-0.2 -0.18 -0.08 rpy=0 0 0

Commit message: Robot positioning and arms fixed

File: ball_pusher_robot/urdf/ball_pusher_with_physics.urdf (robot description, URDF)
Before this commit: robot ball_pusher, 11 links, 10 joints
Joints:
- joint left_arm_joint: limit lower=-1.2 upper=0.3 effort=10 velocity=1 -> (none); type revolute -> fixed
- joint right_arm_joint: limit lower=-1.2 upper=0.3 effort=10 velocity=1 -> (none); type revolute -> fixed
